File: hardware/CAM-M8Q-Breakout_v10.brd (EAGLE design)
At the start: 37 x 28 mm, 20 parts, among them J2 MA06-1, J3 MA06-1, X1 PASSER-07, X2 PASSER-07, X3 PASSER-07, X4 PASSER-07

Commit message: updated layout and schematics
Parts:
- removed J3: MA06-1, we-con:MA06-1
- added J1: MA06-1, we-con:MA06-1
- R1, R2: value (none) -> nc
- R3: value (none) -> 0
- moved J2 15.7 mm to (24.7, 2.00), turned to 90 degrees
Connections:
- net EXT_INT: now also J2.5; no longer J3.5
- net GND: now also J1.2; no longer J2.2
- net LNA_EN: now also J2.4; no longer J3.4
- net RESET: now also J2.2; no longer J3.2
- net RXD: now also J1.4; no longer J2.4
- net SAFEBOOT: now also J2.3; no longer J3.3
- net SCL: now also J1.5; no longer J2.5
- net SDA: now also J1.6; no longer J2.6
- net TIMEPULS: now also J2.6; no longer J3.6
- net TXD: now also J1.3; no longer J2.3
- net VCC: now also J1.1; no longer J2.1
- net VIO: now also J2.1; no longer J3.1
Changed lines of the file:
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@@
 <attribute name="NAME" x="13.08125" y="5.31775" size="0.8128" layer="21" font="vector" ratio="14" rot="R180" align="center"/>
 </element>
-<element name="J2" library="we-con" package="MA06-1" value="MA06-1" x="34.877" y="14" smashed="yes"/>
-<element name="J3" library="we-con" package="MA06-1" value="MA06-1" x="24.717" y="2" smashed="yes" rot="R90"/>
+<element name="J1" library="we-con" package="MA06-1" value="MA06-1" x="34.877" y="14" smashed="yes"/>
+<element name="J2" library="we-con" package="MA06-1" value="MA06-1" x="24.717" y="2" smashed="yes" rot="R90"/>
 <element name="VCC-VIO" library="we-rcl" package="JUMPER2-0603_NC" value="JUMPER2-0603-NC" x="11.1445" y="22.27225" smashed="yes" rot="R90">
 <attribute name="NAME" x="12.5415" y="20.8435" size="0.8128" layer="21" font="vector" ratio="14" rot="R180" align="center"/>
@@
 <attribute name="VALUE" x="8.715" y="12.825" size="0.8128" layer="27" font="vector" ratio="10" align="center"/>
 </element>
-<element name="R1" library="we-rcl" package="C0402" value="" x="5.921" y="7.142" smashed="yes" rot="R180">
+<element name="R1" library="we-rcl" package="C0402" value="nc" x="5.921" y="7.142" smashed="yes" rot="R180">
 <attribute name="NAME" x="6.937" y="7.142" size="0.6096" layer="25" font="vector" ratio="14" rot="R90" align="center"/>
 <attribute name="VALUE" x="4.651" y="7.142" size="0.8128" layer="27" font="vector" ratio="10" rot="R90" align="center"/>
 </element>
-<element name="R2" library="we-rcl" package="C0402" value="" x="4.905" y="7.142" smashed="yes" rot="R180">
+<element name="R2" library="we-rcl" package="C0402" value="nc" x="4.905" y="7.142" smashed="yes" rot="R180">
 <attribute name="NAME" x="3.889" y="7.142" size="0.6096" layer="25" font="vector" ratio="14" rot="R90" align="center"/>
 <attribute name="VALUE" x="3.635" y="7.142" size="0.8128" layer="27" font="vector" ratio="10" rot="R90" align="center"/>
 </element>
-<element name="R3" library="we-rcl" package="C0402" value="" x="5.413" y="7.65" smashed="yes" rot="R270">
+<element name="R3" library="we-rcl" package="C0402" value="0" x="5.413" y="7.65" smashed="yes" rot="R270">
 <attribute name="NAME" x="5.413" y="8.412" size="0.6" layer="25" font="vector" ratio="14" rot="R180" align="center"/>
 <attribute name="VALUE" x="5.413" y="6.38" size="0.8128" layer="27" font="vector" ratio="10" rot="R180" align="center"/>
@@
 <contactref element="C1" pad="1"/>
 <contactref element="D_SEL" pad="2"/>
-<contactref element="J2" pad="2"/>
+<contactref element="J1" pad="2"/>
 <contactref element="GPS" pad="27"/>
 <contactref element="GPS" pad="11"/>
@@
 <contactref element="VCC-VIO" pad="1"/>
 <contactref element="C1" pad="2"/>
-<contactref element="J2" pad="1"/>
+<contactref element="J1" pad="1"/>
 <contactref element="GPS" pad="9"/>
 <wire x1="6.915" y1="18.4" x2="6.915" y2="19.89" width="0.4064" layer="1"/>
@@
 </signal>
 <signal name="TXD">
-<contactref element="J2" pad="3"/>
+<contactref element="J1" pad="3"/>
 <contactref element="GPS" pad="25"/>
 <wire x1="34.877" y1="15.27" x2="33.90725" y2="15.27" width="0.4064" layer="1"/>
@@
 </signal>
 <signal name="RXD">
-<contactref element="J2" pad="4"/>
+<contactref element="J1" pad="4"/>
 <contactref element="GPS" pad="26"/>
 <wire x1="34.877" y1="12.73" x2="33.8755" y2="12.73" width="0.4064" layer="1"/>
@@
 </signal>
 <signal name="SCL">
-<contactref element="J2" pad="5"/>
+<contactref element="J1" pad="5"/>
 <contactref element="GPS" pad="6"/>
 <wire x1="34.877" y1="10.19" x2="33.97075" y2="10.19" width="0.4064" layer="1"/>
@@
 </signal>
 <signal name="SDA">
-<contactref element="J2" pad="6"/>
+<contactref element="J1" pad="6"/>
 <contactref element="GPS" pad="3"/>
 <wire x1="34.877" y1="7.65" x2="33.879" y2="7.65" width="0.4064" layer="1"/>
@@
 <signal name="RESET">
 <contactref element="GPS" pad="23"/>
-<contactref element="J3" pad="2"/>
+<contactref element="J2" pad="2"/>
 <wire x1="11.915" y1="9.6" x2="11.915" y2="8.659" width="0.254" layer="1"/>
 <wire x1="11.915" y1="8.659" x2="12.7" y2="7.874" width="0.254" layer="1"/>
@@
 <signal name="SAFEBOOT">
 <contactref element="GPS" pad="24"/>
-<contactref element="J3" pad="3"/>
+<contactref element="J2" pad="3"/>
 <wire x1="12.915" y1="9.6" x2="12.915" y2="8.675" width="0.254" layer="1"/>
 <wire x1="12.915" y1="8.675" x2="13.208" y2="8.382" width="0.254" layer="1"/>
@@
 <signal name="LNA_EN">
 <contactref element="GPS" pad="30"/>
-<contactref element="J3" pad="4"/>
+<contactref element="J2" pad="4"/>
 <wire x1="25.987" y1="2" x2="25.987" y2="9.446" width="0.254" layer="16"/>
 <via x="20.574" y="14.859" extent="1-16" drill="0.3"/>
@@
 <signal name="EXT_INT">
 <contactref element="GPS" pad="7"/>
-<contactref element="J3" pad="5"/>
+<contactref element="J2" pad="5"/>
 <wire x1="28.527" y1="2" x2="28.527" y2="11.95425" width="0.254" layer="16"/>
 <wire x1="19.2405" y1="21.2725" x2="19.20875" y2="21.2725" width="0.254" layer="16"/>
@@
 <signal name="TIMEPULS">
 <contactref element="GPS" pad="29"/>
-<contactref element="J3" pad="6"/>
+<contactref element="J2" pad="6"/>
 <wire x1="31.067" y1="2" x2="31.067" y2="12.621" width="0.254" layer="16"/>
 <via x="29.718" y="13.97" extent="1-16" drill="0.3"/>
@@
 <contactref element="GPS" pad="1"/>
 <contactref element="VCC-VIO" pad="2"/>
-<contactref element="J3" pad="1"/>
+<contactref element="J2" pad="1"/>
 <wire x1="18.367" y1="2" x2="18.367" y2="3.127" width="0.254" layer="16"/>
 <via x="18.923" y="18.415" extent="1-16" drill="0.3"/>
